Commit message: tweaks

File: kortex_description/arms/gen3_lite/6dof/urdf/GEN3-LITE.urdf (robot description, URDF)
Before this commit: robot KR7108-URDF, 8 links, 7 joints
Links:
- link ARM: geometry collision mesh filename=package://kortex_description/gen3_lite/meshes/arm_link.STL; visual mesh filename=package://kortex_description/gen3_lite/meshes/arm_link.STL
- link BASE: geometry collision mesh filename=package://kortex_description/gen3_lite/meshes/base_link.STL; visual mesh filename=package://kortex_description/gen3_lite/meshes/base_link.STL
- link FOREARM: geometry collision mesh filename=package://kortex_description/gen3_lite/meshes/forearm_link.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; visual mesh filename=package://kortex_description/gen3_lite/meshes/forearm_link.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
- link LOWER_WRIST: geometry collision mesh filename=package://kortex_description/gen3_lite/meshes/lower_wrist_l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; visual mesh filename=package://kortex_description/gen3_lite/meshes/lower_wrist_l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
- link SHOULDER: geometry collision mesh filename=package://kortex_description/gen3_lite/meshes/shoulder_link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; visual mesh filename=package://kortex_description/gen3_lite/meshes/shoulder_link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
- link UPPER_WRIST: geometry collision mesh filename=package://kortex_description/gen3_lite/meshes/upper_wrist_l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; visual mesh filename=package://kortex_description/gen3_lite/meshes/upper_wrist_l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

File: kortex_description/grippers/gen3_lite_2f/urdf/GEN3-LITE-GRIPPER_URDF_SIMPLIFIED_V2.urdf (robot description, URDF)
Before this commit: robot L31K-GRIPPER_URDF_SIMPLIFIED_V2, 5 links, 4 joints
Joints:
- joint LEFT_BOTTOM: limit lower=-0.96 upper=0.09 effort=1000 velocity=1000 -> lower=-0.96 upper=0.09 effort=10 velocity=1000
- joint LEFT_TIP: limit lower=-0.21 upper=1.03 effort=1000 velocity=1000 -> lower=-0.21 upper=1.03 effort=10 velocity=1000
- joint RIGHT_BOTTOM: limit lower=-0.09 upper=0.96 effort=1000 velocity=1000 -> lower=-0.09 upper=0.96 effort=10 velocity=1000
- joint RIGHT_TIP: limit lower=-1.03 upper=0.21 effort=1000 velocity=1000 -> lower=-1.03 upper=0.21 effort=10 velocity=1000

File: kortex_description/grippers/gen3_lite_2f/urdf/gen3_lite_2f_macro.xacro (robot description, xacro)
@@ -72,5 +72,6 @@
       <child link="${prefix}right_finger_prox_link" />
       <axis xyz="0 0 1" />
-      <limit lower="-0.09" upper="0.96" effort="1000" velocity="0.6" />
+      <!-- <limit lower="-0.09" upper="0.96" effort="10" velocity="0.6" /> -->
+      <limit lower="-0.09" upper="0.96" effort="10" velocity="0.2" />
     </joint>
     <link name="${prefix}right_finger_dist_link">
@@ -104,5 +105,6 @@
       <child link="${prefix}right_finger_dist_link" />
       <axis xyz="0 0 1" />
-      <limit lower="-0.50" upper="0.21" effort="1000" velocity="1000" /> <!--limit lower="-1.03" upper="0.21" effort="1000" velocity="1000" /-->
+      <!-- <limit lower="-0.50" upper="0.21" effort="10" velocity="1000" /> limit lower="-1.03" upper="0.21" effort="1000" velocity="1000" / -->
+      <limit lower="-0.50" upper="0.21" effort="10" velocity="1000" /> <!--limit lower="-1.03" upper="0.21" effort="1000" velocity="1000" /-->
       <mimic joint="${prefix}right_finger_bottom_joint" multiplier="-0.676" offset="0.149" />
     </joint>
@@ -137,5 +139,6 @@
       <child link="${prefix}left_finger_prox_link" />
       <axis xyz="0 0 1" />
-      <limit lower="-0.96" upper="0.09" effort="1000" velocity="1000" />
+      <!-- <limit lower="-0.96" upper="0.09" effort="10" velocity="1000" /> -->
+      <limit lower="-0.96" upper="0.09" effort="10" velocity="1000" />
       <mimic joint="${prefix}right_finger_bottom_joint" multiplier="-1.0" offset="0.0" />
     </joint>
@@ -170,7 +173,109 @@
       <child link="${prefix}left_finger_dist_link" />
       <axis xyz="0 0 -1" />
-      <limit lower="-0.50" upper="0.21" effort="1000" velocity="1000" /> <!--limit lower="-1.03" upper="0.21" effort="1000" velocity="1000" /-->
+      <!-- <limit lower="-0.50" upper="0.21" effort="10" velocity="1000" /> limit lower="-1.03" upper="0.21" effort="1000" velocity="1000" / -->
+      <limit lower="-0.50" upper="0.21" effort="10" velocity="1000" /> <!--limit lower="-1.03" upper="0.21" effort="1000" velocity="1000" /-->
       <mimic joint="${prefix}right_finger_bottom_joint" multiplier="-0.676" offset="0.149" />
     </joint>
+    <!-- Add friction -->
+    <gazebo reference="${prefix}right_finger_prox_link">
+    <collision name="${prefix}right_finger_prox_link_collision">
+      <surface>
+        <friction>
+          <torsional>
+            <coefficient>10.0</coefficient>
+            <use_patch_radius>true</use_patch_radius>
+            <patch_radius>0.05</patch_radius>
+          </torsional>
+        </friction>
+        <contact>
+          <poissons_ratio>0.5</poissons_ratio>
+          <elastic_modulus>1e8</elastic_modulus>
+        </contact>
+      </surface>
+    </collision>
+    <mu1>100</mu1>
+    <mu2>100</mu2>
+    <maxVel>1</maxVel>
+    <kp>1000000.0</kp>
+    <kd>100.0</kd>
+    <fdir1>0 0 1</fdir1>
+    <minDepth>0.0</minDepth>
+    <maxContacts>100</maxContacts>
+  </gazebo>
+  <gazebo reference="${prefix}right_finger_dist_link">
+    <collision name="${prefix}right_finger_dist_link_collision">
+      <surface>
+        <friction>
+          <torsional>
+            <coefficient>10.0</coefficient>
+            <use_patch_radius>true</use_patch_radius>
+            <patch_radius>0.05</patch_radius>
+          </torsional>
+        </friction>
+        <contact>
+          <poissons_ratio>0.5</poissons_ratio>
+          <elastic_modulus>1e8</elastic_modulus>
+        </contact>
+      </surface>
+    </collision>
+    <mu1>100</mu1>
+    <mu2>100</mu2>
+    <maxVel>1</maxVel>
+    <kp>1000000.0</kp>
+    <kd>100.0</kd>
+    <fdir1>0 0 1</fdir1>
+    <minDepth>0.0</minDepth>
+    <maxContacts>100</maxContacts>
+  </gazebo>
+  <gazebo reference="${prefix}left_finger_prox_link">
+    <collision name="${prefix}left_finger_prox_link_collision">
+      <surface>
+        <friction>
+          <torsional>
+            <coefficient>10.0</coefficient>
+            <use_patch_radius>true</use_patch_radius>
+            <patch_radius>0.05</patch_radius>
+          </torsional>
+        </friction>
+        <contact>
+          <poissons_ratio>0.5</poissons_ratio>
+          <elastic_modulus>1e8</elastic_modulus>
+        </contact>
+      </surface>
+    </collision>
+    <mu1>100</mu1>
+    <mu2>100</mu2>
+    <maxVel>1</maxVel>
+    <kp>1000000.0</kp>
+    <kd>100.0</kd>
+    <fdir1>0 0 1</fdir1>
+    <minDepth>0.0</minDepth>
+    <maxContacts>100</maxContacts>
+  </gazebo>
+  <gazebo reference="${prefix}left_finger_dist_link">
+    <collision name="${prefix}left_finger_dist_link_collision">
+      <surface>
+        <friction>
+          <torsional>
+            <coefficient>10.0</coefficient>
+            <use_patch_radius>true</use_patch_radius>
+            <patch_radius>0.05</patch_radius>
+          </torsional>
+        </friction>
+        <contact>
+          <poissons_ratio>0.5</poissons_ratio>
+          <elastic_modulus>1e8</elastic_modulus>
+        </contact>
+      </surface>
+    </collision>
+    <mu1>100</mu1>
+    <mu2>100</mu2>
+    <maxVel>1</maxVel>
+    <kp>1000000.0</kp>
+    <kd>100.0</kd>
+    <fdir1>0 0 1</fdir1>
+    <minDepth>0.0</minDepth>
+    <maxContacts>100</maxContacts>
+  </gazebo>
   </xacro:macro>
 </robot>

File: kortex_description/grippers/gen3_lite_2f/urdf/gen3_lite_2f_transmission_macro.xacro (robot description, xacro)
@@ -6,8 +6,10 @@
             <joint name="${prefix}right_finger_bottom_joint">
                 <hardwareInterface>hardware_interface/PositionJointInterface</hardwareInterface>
+                <!-- <hardwareInterface>hardware_interface/EffortJointInterface</hardwareInterface> -->
             </joint>
             <actuator name="${prefix}right_finger_bottom_motor">
                 <mechanicalReduction>1</mechanicalReduction>
                 <hardwareInterface>hardware_interface/PositionJointInterface</hardwareInterface>
+                <!-- <hardwareInterface>hardware_interface/EffortJointInterface</hardwareInterface> -->
             </actuator>
         </transmission>
@@ -42,12 +44,14 @@
                     <palm_link>${prefix}end_effector_link</palm_link> <!-- Gazebo merges links connected by fixed joints, so here we would have put gripper_base_link but it is merged with Bracelet_Link internally -->
                     <gripper_link> ${prefix}right_finger_dist_link </gripper_link>
+                    <gripper_link> ${prefix}right_finger_prox_link </gripper_link>
                     <gripper_link> ${prefix}left_finger_dist_link </gripper_link>
+                    <gripper_link> ${prefix}left_finger_prox_link </gripper_link>
                 </arm>
                 <forces_angle_tolerance>100</forces_angle_tolerance>
                 <update_rate>10</update_rate>
-                <grip_count_threshold>3</grip_count_threshold>
+                <grip_count_threshold>2</grip_count_threshold>
                 <max_grip_count>10</max_grip_count>
-                <release_tolerance>0.001</release_tolerance>
-                <disable_collisions_on_attach>false</disable_collisions_on_attach>
+                <release_tolerance>0.005</release_tolerance>
+                <disable_collisions_on_attach>true</disable_collisions_on_attach>
                 <contact_topic>__default_topic__</contact_topic>
             </plugin>

File: kortex_move_it_config/gen3_lite_gen3_lite_2f_move_it_config/config/gen3_lite_gen3_lite_2f.srdf.xacro (robot description, xacro)
@@ -66,5 +66,6 @@
     </group_state>
     <!--END EFFECTOR: Purpose: Represent information about an end effector.-->
-    <end_effector name="end_effector" parent_link="$(arg prefix)tool_frame" group="arm" />
+    <!-- <end_effector name="end_effector" parent_link="$(arg prefix)tool_frame" group="arm" /> -->
+    <end_effector name="end_effector" parent_link="$(arg prefix)dummy_link" group="gripper" parent_group="arm" />
     <!--PASSIVE JOINT: Purpose: this element is used to mark joints that are not actuated-->
     <passive_joint name="$(arg prefix)right_finger_tip_joint" />
